File: type-c_splitter.kicad_sch (KiCad schematic)
At the start: 5 parts, among them J1 Power, J2 Data, P1 Plug

Commit message: Add pdf and step
Changed lines of the file:
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@@
+    (stroke (width 0) (type solid) (color 0 0 0 0))
+  )
+  (wire (pts (xy 157.48 189.23) (xy 157.48 190.5))
+    (stroke (width 0) (type solid) (color 0 0 0 0))
+  )
+  (wire (pts (xy 167.64 189.23) (xy 167.64 190.5))
     (stroke (width 0) (type solid) (color 0 0 0 0))
   )
@@
   (wire (pts (xy 198.12 114.3) (xy 198.12 113.03))
     (stroke (width 0) (type solid) (color 0 0 0 0))
+  )
+  (symbol (lib_id "power:PWR_FLAG") (at 157.48 190.5 180) (unit 1)
+    (in_bom yes) (on_board yes)
+    (property "Reference" "#FLG0102" (id 0) (at 157.48 192.405 0)
+      (effects (font (size 1.27 1.27)) hide)
+    )
+    (property "Value" "PWR_FLAG" (id 1) (at 157.48 194.31 0))
+    (property "Footprint" "" (id 2) (at 157.48 190.5 0)
+      (effects (font (size 1.27 1.27)) hide)
+    )
+    (property "Datasheet" "~" (id 3) (at 157.48 190.5 0)
+      (effects (font (size 1.27 1.27)) hide)
+    )
+    (pin "1")
+  )
+  (symbol (lib_id "power:PWR_FLAG") (at 167.64 189.23 0) (unit 1)
+    (in_bom yes) (on_board yes)
+    (property "Reference" "#FLG0101" (id 0) (at 167.64 187.325 0)
+      (effects (font (size 1.27 1.27)) hide)
+    )
+    (property "Value" "PWR_FLAG" (id 1) (at 167.64 185.42 0))
+    (property "Footprint" "" (id 2) (at 167.64 189.23 0)
+      (effects (font (size 1.27 1.27)) hide)
+    )
+    (property "Datasheet" "~" (id 3) (at 167.64 189.23 0)
+      (effects (font (size 1.27 1.27)) hide)
+    )
+    (pin "1")
   )
   (symbol (lib_id "power:VBUS") (at 113.03 34.29 0) (unit 1)
@@
     (pin "1")
   )
+  (symbol (lib_id "power:VBUS") (at 157.48 189.23 0) (unit 1)
+    (in_bom yes) (on_board yes)
+    (property "Reference" "#PWR0109" (id 0) (at 157.48 193.04 0)
+      (effects (font (size 1.27 1.27)) hide)
+    )
+    (property "Value" "VBUS" (id 1) (at 157.48 185.42 0))
+    (property "Footprint" "" (id 2) (at 157.48 189.23 0)
+      (effects (font (size 1.27 1.27)) hide)
+    )
+    (property "Datasheet" "" (id 3) (at 157.48 189.23 0)
+      (effects (font (size 1.27 1.27)) hide)
+    )
+    (pin "1")
+  )
   (symbol (lib_id "power:VBUS") (at 173.99 73.66 0) (unit 1)
     (in_bom yes) (on_board yes)
@@
     )
     (property "Datasheet" "" (id 3) (at 124.46 43.18 0)
+      (effects (font (size 1.27 1.27)) hide)
+    )
+    (pin "1")
+  )
+  (symbol (lib_id "power:GND") (at 167.64 190.5 0) (unit 1)
+    (in_bom yes) (on_board yes)
+    (property "Reference" "#PWR0110" (id 0) (at 167.64 196.85 0)
+      (effects (font (size 1.27 1.27)) hide)
+    )
+    (property "Value" "GND" (id 1) (at 167.64 194.31 0))
+    (property "Footprint" "" (id 2) (at 167.64 190.5 0)
+      (effects (font (size 1.27 1.27)) hide)
+    )
+    (property "Datasheet" "" (id 3) (at 167.64 190.5 0)
       (effects (font (size 1.27 1.27)) hide)
     )
@@
   )
   (symbol_instances
+    (path "/0c606397-aee5-4a40-9132-52ece525676a"
+      (reference "#FLG0101") (unit 1) (value "PWR_FLAG") (footprint "")
+    )
+    (path "/5d30296e-25d9-4288-9943-b73907804297"
+      (reference "#FLG0102") (unit 1) (value "PWR_FLAG") (footprint "")
+    )
     (path "/da45f0f9-ff33-4dc7-9b41-62fa7781522e"
       (reference "#PWR0101") (unit 1) (value "GND") (footprint "")
@@
       (reference "#PWR0108") (unit 1) (value "VBUS") (footprint "")
     )
+    (path "/f1957df9-6c64-48f4-8f68-50fbf38435b4"
+      (reference "#PWR0109") (unit 1) (value "VBUS") (footprint "")
+    )
+    (path "/ecb40b2e-d88f-4916-977f-b5bde102189b"
+      (reference "#PWR0110") (unit 1) (value "GND") (footprint "")
+    )
     (path "/23d9cb3a-a37e-400d-af22-c79cb4c39b83"
