File: type-c_splitter.kicad_pcb (KiCad board)
At the start: 2 copper layers, 21 x 28 mm, 10 parts, among them J1 Power, J2 Data, P1 Plug

Commit message: Add pdf and step
Connections:
- J1 pad A6: unconnected-(J1-PadA6) -> (no net)
- J1 pad A7: unconnected-(J1-PadA7) -> (no net)
- J1 pad A8: unconnected-(J1-PadA8) -> (no net)
- J1 pad B6: unconnected-(J1-PadB6) -> (no net)
- J1 pad B7: unconnected-(J1-PadB7) -> (no net)
- J1 pad B8: unconnected-(J1-PadB8) -> (no net)
- J2 pad A8: unconnected-(J2-PadA8) -> (no net)
- J2 pad B8: unconnected-(J2-PadB8) -> (no net)

Commit message: Add JLCJLCJLCJLC
Other:
- board text added: "JLCJLCJLCJLC"
Changed lines of the file:
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@@
     (effects (font (size 0.8 0.8) (thickness 0.12)) (justify mirror))
+  )
+  (gr_text "JLCJLCJLCJLC" (at 151 72.5 -90) (layer "F.SilkS")
+    (effects (font (size 0.85 0.85) (thickness 0.15)))
   )
   (dimension (type aligned) (layer "Margin")
